File: adc1283/adc1283.kicad_sch (KiCad schematic)
At the start: 25 parts, among them J1 ToADC, J2 Sensors, U3 MIC5366-2.0YC5-TR

Commit message: board revs, updated README
Parts:
- removed C1, C6: 1uF X7R, Capacitor_SMD:C_0805_2012Metric, symbol Device:C_Small
- removed C3: 10nF NP0, Capacitor_SMD:C_0805_2012Metric, symbol Device:C_Small
- removed H1, H2: MountingHole, MountingHole:MountingHole_3.2mm_M3, symbol Mechanical:MountingHole
- removed J2: Sensors, Connector_PinSocket_2.54mm:PinSocket_2x08_P2.54mm_Vertical, symbol Connector_Generic:Conn_02x08_Odd_Even
- removed R1, R2, R3, R4, R5, R6, R7, R8: 1k, Resistor_SMD:R_0805_2012Metric, symbol Device:R_Small_US
- removed TP1, TP2, TP3, TP4, TP5, TP6, TP7, TP8: TestPoint, TestPoint:TestPoint_Pad_D2.0mm, symbol Connector:TestPoint
- removed U3: MIC5366-2.0YC5-TR, Package_TO_SOT_SMD:SOT-353_SC-70-5, symbol Regulator_Linear:APE8865U5-20-HF-3
- added C1, C3: 4.7uF, Capacitor_SMD:C_0805_2012Metric, symbol Device:C_Polarized_US
- added C13: 100nF, Capacitor_SMD:C_0805_2012Metric, symbol Device:C_Small
- added C4: 1uF, Capacitor_SMD:C_0805_2012Metric, symbol Device:C_Small
- added FB1: FB, Inductor_SMD:L_0805_2012Metric, symbol Device:FerriteBead_Small
- added J2: Conn_01x20, Connector_PinHeader_2.54mm:PinHeader_2x10_P2.54mm_Vertical, symbol Connector_Generic:Conn_01x20
- added JP1: VDirect, Jumper:SolderJumper-2_P1.3mm_Open_RoundedPad1.0x1.5mm, symbol Jumper:Jumper_2_Open
- added U2: LT1963AxST-3.3, Package_TO_SOT_SMD:SOT-223-3_TabPin2, symbol Regulator_Linear:LT1963AxST-3.3
- added U3: ADC1283, Package_SO:TSSOP-16_4.4x5mm_P0.65mm, symbol Analog_ADC:ADC1283
- C2: value 1uF X7R -> 1uF
- J1: value ToADC -> Glasgow; footprint Connector_PinSocket_2.54mm:PinSocket_2x10_P2.54mm_Vertical -> Connector_PinHeader_2.54mm:PinHeader_2x10_P2.54mm_Vertical; DigiKey (none) -> SSW-110-03-T-D-ND
Connections:
- net GND: now also J1.10 (Pin_10), J1.12 (Pin_12), J1.14 (Pin_14), J1.16 (Pin_16), J1.4 (Pin_4), J1.6 (Pin_6), J1.8 (Pin_8), C1.2, C13.2, C3.2, C4.2, J2.17 (Pin_17), J2.19 (Pin_19), U2.2 (GND), U3.12 (DGND), U3.3 (AGND); no longer J1.20 (Pin_20)
- net VAA: now also C3.1, C4.1, FB1.1, J2.20 (Pin_20); no longer C2.1, J1.19 (Pin_19)
- net S0: no longer names the net of J1.1 (Pin_1)
- net S1: no longer names the net of J1.3 (Pin_3)
- net S2: no longer names the net of J1.5 (Pin_5)
- net S3 renamed MOSI
- net MOSI: now also U3.14 (DIN)
- net S4 renamed MISO
- net MISO: now also U3.15 (DOUT)
- net S5 renamed SCLK
- net SCLK: now also U3.16 (SCLK)
- net S6: no longer names the net of J1.13 (Pin_13)
- net S7 renamed ~{CS}
- net ~{CS}: now also U3.1 (~{CS})
- removed net VREF: J1.10 (Pin_10), J1.12 (Pin_12), J1.14 (Pin_14), J1.16 (Pin_16), J1.17 (Pin_17), J1.2 (Pin_2), J1.4 (Pin_4), J1.6 (Pin_6), J1.8 (Pin_8)
- new net: FB1.2, JP1.2 (B), U2.3 (OUT)
- new net AIN0N: J2.2 (Pin_2), U3.4 (IN0)
- new net AIN1N: J2.4 (Pin_4), U3.5 (IN1)
- new net AIN2N: J2.6 (Pin_6), U3.6 (IN2)
- new net AIN3N: J2.8 (Pin_8), U3.7 (IN3)
- new net AIN4N: J2.10 (Pin_10), U3.8 (IN4)
- new net AIN5N: J2.12 (Pin_12), U3.9 (IN5)
- new net AIN6N: J2.14 (Pin_14), U3.10 (IN6)
- new net AIN7N: J2.16 (Pin_16), U3.11 (IN7)
- new net VDD: C1.1, C2.1, J1.20 (Pin_20), JP1.1 (A), U2.1 (IN), U3.13 (DVCC)
- new net VREFIN: C13.1, J2.18 (Pin_18), U3.2 (AVCC)
- no-connect marks 1 -> 15
Other:
- note added: "IO0"
- note added: "IO1"
- note added: "IO2"
- note added: "IO3"
- note added: "IO4"
- note added: "IO5"
- note added: "IO6"
- note added: "IO7"
- note added: "SamTec SSW-110-03-T-D should mate with Glasgow, and have posts sticking up"
- note added: "Sense"
- note added: "capacitance covered by C1,C3,C4"
- note removed: "Also: REF3312AIDCKR 1.25V, lower noise $1.76/ea @ 10"
- note removed: "NP0 GRM2165C2A103JA01D"
