File: ads131m08/ads131m08.kicad_pcb (KiCad board)
At the start: 4 copper layers, 63.5 x 37.5 mm, 22 parts, among them J1 Glasgow, J2 Conn_01x20, U1 ADS131M08

Commit message: board revs, updated README
Connections:
- J1 pad 2: VDD -> unconnected-(J1-Pin_2-Pad2)
- J1 pad 20: unconnected-(J1-Pin_20-Pad20) -> VDD
Other:
- board text added: "glasgow interface rev1"
- board text removed: "glasgow interface rev0"
