File: ads131m08/ads131m08.kicad_sch (KiCad schematic)
At the start: 22 parts, among them J1 Glasgow, J2 Conn_01x20, U1 ADS131M08

Commit message: board revs, updated README
Connections:
- net VDD: now also J1.20 (Pin_20); no longer J1.2 (Pin_2)
Changed lines of the file:
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@@
 	)
 	(junction
-		(at 231.14 80.01)
+		(at 96.52 73.66)
 		(diameter 0)
 		(color 0 0 0 0)
 	)
 	(junction
-		(at 96.52 73.66)
+		(at 231.14 80.01)
 		(diameter 0)
 		(color 0 0 0 0)
@@
 	)
 	(no_connect
-		(at 168.91 109.22)
+		(at 215.9 100.33)
 	)
 	(no_connect
-		(at 215.9 80.01)
+		(at 168.91 109.22)
 	)
 	(no_connect
-		(at 215.9 82.55)
+		(at 215.9 80.01)
 	)
 	(no_connect
@@
 	(wire
 		(pts
-			(xy 199.39 87.63) (xy 215.9 87.63)
+			(xy 199.39 85.09) (xy 215.9 85.09)
 		)
 		(stroke
@@
 	(wire
 		(pts
-			(xy 199.39 100.33) (xy 215.9 100.33)
+			(xy 199.39 97.79) (xy 215.9 97.79)
 		)
 		(stroke
@@
 	(wire
 		(pts
-			(xy 228.6 80.01) (xy 231.14 80.01)
+			(xy 125.73 90.17) (xy 96.52 90.17)
 		)
 		(stroke
@@
 	(wire
 		(pts
-			(xy 125.73 90.17) (xy 96.52 90.17)
+			(xy 199.39 90.17) (xy 215.9 90.17)
 		)
 		(stroke
@@
 	(wire
 		(pts
-			(xy 199.39 92.71) (xy 215.9 92.71)
+			(xy 64.77 95.25) (xy 78.74 95.25)
 		)
 		(stroke
@@
 	(wire
 		(pts
-			(xy 64.77 95.25) (xy 78.74 95.25)
+			(xy 33.02 111.76) (xy 35.56 111.76)
 		)
 		(stroke
@@
 	(wire
 		(pts
-			(xy 33.02 111.76) (xy 35.56 111.76)
+			(xy 64.77 80.01) (xy 78.74 80.01)
 		)
 		(stroke
@@
 	(wire
 		(pts
-			(xy 64.77 80.01) (xy 78.74 80.01)
+			(xy 97.79 87.63) (xy 97.79 80.01)
 		)
 		(stroke
@@
 	(wire
 		(pts
-			(xy 97.79 87.63) (xy 97.79 80.01)
+			(xy 228.6 80.01) (xy 231.14 80.01)
 		)
 		(stroke
@@
 	(wire
 		(pts
-			(xy 199.39 97.79) (xy 215.9 97.79)
+			(xy 199.39 95.25) (xy 215.9 95.25)
 		)
 		(stroke
@@
 	(wire
 		(pts
-			(xy 199.39 90.17) (xy 215.9 90.17)
+			(xy 199.39 87.63) (xy 215.9 87.63)
 		)
 		(stroke
@@
 	(wire
 		(pts
-			(xy 199.39 85.09) (xy 215.9 85.09)
+			(xy 199.39 82.55) (xy 215.9 82.55)
 		)
 		(stroke
@@
 	(wire
 		(pts
-			(xy 199.39 95.25) (xy 215.9 95.25)
+			(xy 199.39 92.71) (xy 215.9 92.71)
 		)
 		(stroke
@@
 	(text "IO3"
 		(exclude_from_sim no)
-		(at 213.36 89.408 0)
+		(at 213.36 91.948 0)
 		(effects
 			(font
@@
 	(text "IO6"
 		(exclude_from_sim no)
-		(at 213.36 97.028 0)
+		(at 213.36 84.328 0)
 		(effects
 			(font
@@
 	(text "IO5"
 		(exclude_from_sim no)
-		(at 213.36 94.488 0)
+		(at 213.36 86.868 0)
 		(effects
 			(font
@@
 	(text "Sense\n"
 		(exclude_from_sim no)
-		(at 212.344 79.248 0)
+		(at 212.09 79.502 0)
 		(effects
 			(font
@@
 	(text "IO7\n"
 		(exclude_from_sim no)
-		(at 213.36 99.568 0)
+		(at 213.36 81.788 0)
 		(effects
 			(font
@@
 	(text "IO2"
 		(exclude_from_sim no)
-		(at 213.36 86.868 0)
+		(at 213.36 94.488 0)
 		(effects
 			(font
@@
 	(text "IO4"
 		(exclude_from_sim no)
-		(at 213.36 91.948 0)
+		(at 213.36 89.408 0)
 		(effects
 			(font
@@
 	(text "IO1"
 		(exclude_from_sim no)
-		(at 213.36 84.328 0)
+		(at 213.36 97.028 0)
 		(effects
 			(font
@@
 	(text "IO0"
 		(exclude_from_sim no)
-		(at 213.36 81.788 0)
+		(at 213.36 99.568 0)
 		(effects
 			(font
@@
 	)
 	(label "~{DRDY}"
-		(at 170.18 97.79 0)
+		(at 176.53 97.79 180)
 		(fields_autoplaced yes)
 		(effects
@@
 				(size 1.27 1.27)
 			)
-			(justify left bottom)
+			(justify right bottom)
 		)
 	)
@@
 	)
 	(label "~{DRDY}"
-		(at 199.39 95.25 0)
+		(at 199.39 87.63 0)
 		(fields_autoplaced yes)
 		(effects
@@
 	)
 	(label "~{CS}"
-		(at 199.39 97.79 0)
+		(at 199.39 85.09 0)
 		(fields_autoplaced yes)
 		(effects
@@
 	)
 	(label "MISO"
-		(at 199.39 90.17 0)
+		(at 199.39 92.71 0)
 		(fields_autoplaced yes)
 		(effects
@@
 	)
 	(label "~{CS}"
-		(at 170.18 87.63 0)
+		(at 176.53 87.63 180)
 		(fields_autoplaced yes)
 		(effects
@@
 				(size 1.27 1.27)
 			)
-			(justify left bottom)
+			(justify right bottom)
 		)
 	)
@@
 	)
 	(label "CLKIN"
-		(at 170.18 106.68 0)
+		(at 176.53 106.68 180)
 		(fields_autoplaced yes)
 		(effects
@@
 				(size 1.27 1.27)
 			)
-			(justify left bottom)
+			(justify right bottom)
 		)
 	)
 	(label "SCLK"
-		(at 199.39 92.71 0)
+		(at 199.39 90.17 0)
 		(fields_autoplaced yes)
 		(effects
@@
 	)
 	(label "MOSI"
-		(at 199.39 87.63 0)
+		(at 199.39 95.25 0)
 		(fields_autoplaced yes)
 		(effects
@@
 	)
 	(label "SCLK"
-		(at 170.18 90.17 0)
+		(at 176.53 90.17 180)
 		(fields_autoplaced yes)
 		(effects
@@
 				(size 1.27 1.27)
 			)
-			(justify left bottom)
+			(justify right bottom)
 		)
 	)
@@
 	)
 	(label "MOSI"
-		(at 170.18 92.71 0)
+		(at 176.53 92.71 180)
 		(fields_autoplaced yes)
 		(effects
@@
 				(size 1.27 1.27)
 			)
-			(justify left bottom)
+			(justify right bottom)
 		)
 	)
@@
 	)
 	(label "~{RESET}"
-		(at 170.18 82.55 0)
+		(at 176.53 82.55 180)
 		(fields_autoplaced yes)
 		(effects
@@
 				(size 1.27 1.27)
 			)
-			(justify left bottom)
+			(justify right bottom)
 		)
 	)
@@
 	)
 	(label "CLKIN"
-		(at 199.39 85.09 0)
+		(at 199.39 97.79 0)
 		(fields_autoplaced yes)
 		(effects
@@
 	)
 	(label "~{RESET}"
-		(at 199.39 100.33 0)
+		(at 199.39 82.55 0)
 		(fields_autoplaced yes)
 		(effects
@@
 	)
 	(label "MISO"
-		(at 170.18 95.25 0)
+		(at 176.53 95.25 180)
 		(fields_autoplaced yes)
 		(effects
@@
 				(size 1.27 1.27)
 			)
-			(justify left bottom)
+			(justify right bottom)
 		)
 	)
@@
 	(symbol
 		(lib_id "Connector_Generic:Conn_02x10_Odd_Even")
-		(at 220.98 90.17 0)
+		(at 220.98 92.71 0)
+		(mirror x)
 		(unit 1)
 		(exclude_from_sim no)
@@
 		(on_board yes)
 		(dnp no)
-		(fields_autoplaced yes)
 		(property "Reference" "J1"
-			(at 222.25 74.5955 0)
+			(at 222.25 108.2845 0)
 			(effects
 				(font
@@
 		)
 		(property "Value" "Glasgow"
-			(at 222.25 77.0198 0)
+			(at 222.25 105.8602 0)
 			(effects
 				(font
@@
 		)
 		(property "Footprint" "Connector_PinHeader_2.54mm:PinHeader_2x10_P2.54mm_Vertical"
-			(at 220.98 90.17 0)
+			(at 220.98 92.71 0)
 			(effects
 				(font
@@
 		)
 		(property "Datasheet" "~"
-			(at 220.98 90.17 0)
+			(at 220.98 92.71 0)
 			(effects
 				(font
@@
 		)
 		(property "Description" "Generic connector, double row, 02x10, odd/even pin numbering scheme (row 1 odd numbers, row 2 even numbers), script generated (kicad-library-utils/schlib/autogen/connector/)"
-			(at 220.98 90.17 0)
+			(at 220.98 92.71 0)
 			(effects
 				(font
@@
 		)
 		(property "DigiKey" "SSW-110-03-T-D-ND"
-			(at 220.98 90.17 0)
+			(at 220.98 92.71 0)
 			(effects
 				(font
