File: mcp3008/mcp3008.kicad_pcb (KiCad board)
At the start: 4 copper layers, 63.5 x 37.5 mm, 11 parts, among them J1 Glasgow, J2 Conn_01x20, U1 MCP3008, U2 LT1963AxST-3.3

Commit message: board revs, updated README
Parts:
- added R1: 100k, Resistor_SMD:R_0805_2012Metric, F.Cu at (109.0, 114.2)
Connections:
- J1 pad 2: VDD -> unconnected-(J1-Pin_2-Pad2)
- J1 pad 20: unconnected-(J1-Pin_20-Pad20) -> VDD
Routing:
- net /MISO: track 16.1 -> 19.2 mm, vias 0 -> 2
- net /MOSI: track 21.6 -> 22.3 mm
- net /SCLK: track 19.5 -> 20.1 mm
Other:
- board text added: "glasgow interface rev1"
- board text removed: "glasgow interface rev0"
