File: mcp3008/mcp3008.kicad_sch (KiCad schematic)
At the start: 11 parts, among them J1 Glasgow, J2 Conn_01x20, U1 MCP3008, U2 LT1963AxST-3.3

Commit message: board revs, updated README
Parts:
- added R1: 100k, Resistor_SMD:R_0805_2012Metric, symbol Device:R_Small_US
Connections:
- net MISO: now also R1.2
- net VDD: now also J1.20 (Pin_20), R1.1; no longer J1.2 (Pin_2)
Other:
- note added: "Extremely weak pullup so that when the MCP3008 is don't care, we can distinguish that from the 0 bit that it intentionally sends."
Changed lines of the file:
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@@
+	)
+	(no_connect
+		(at 199.39 100.33)
+	)
+	(no_connect
+		(at 215.9 102.87)
+	)
+	(no_connect
+		(at 82.55 93.98)
+	)
+	(no_connect
+		(at 199.39 87.63)
+	)
+	(no_connect
+		(at 82.55 109.22)
+	)
+	(no_connect
+		(at 82.55 104.14)
+	)
+	(no_connect
+		(at 82.55 83.82)
+	)
+	(no_connect
+		(at 82.55 73.66)
+	)
+	(no_connect
+		(at 215.9 80.01)
+	)
+	(no_connect
+		(at 199.39 97.79)
 	)
 	(no_connect
@@
 	)
 	(no_connect
-		(at 215.9 102.87)
-	)
-	(no_connect
-		(at 82.55 93.98)
-	)
-	(no_connect
-		(at 199.39 95.25)
-	)
-	(no_connect
-		(at 82.55 109.22)
-	)
-	(no_connect
-		(at 82.55 104.14)
-	)
-	(no_connect
-		(at 82.55 83.82)
-	)
-	(no_connect
-		(at 82.55 73.66)
-	)
-	(no_connect
-		(at 215.9 80.01)
-	)
-	(no_connect
-		(at 199.39 85.09)
-	)
-	(no_connect
-		(at 199.39 100.33)
-	)
-	(no_connect
 		(at 82.55 88.9)
 	)
@@
 	(wire
 		(pts
+			(xy 223.52 124.46) (xy 223.52 121.92)
+		)
+		(stroke
+			(width 0)
+			(type default)
+		)
+	)
+	(wire
+		(pts
 			(xy 152.4 76.2) (xy 154.94 76.2)
 		)
@@
 	(wire
 		(pts
+			(xy 223.52 129.54) (xy 223.52 133.35)
+		)
+		(stroke
+			(width 0)
+			(type default)
+		)
+	)
+	(wire
+		(pts
 			(xy 231.14 80.01) (xy 241.3 80.01)
 		)
@@
 	(text "IO3"
 		(exclude_from_sim no)
-		(at 213.36 89.408 0)
+		(at 212.852 89.408 0)
 		(effects
 			(font
@@
 	(text "IO6"
 		(exclude_from_sim no)
-		(at 213.36 97.028 0)
+		(at 212.852 97.028 0)
 		(effects
 			(font
@@
 	(text "IO5"
 		(exclude_from_sim no)
-		(at 213.36 94.488 0)
+		(at 212.852 94.488 0)
 		(effects
 			(font
@@
 	(text "Sense\n"
 		(exclude_from_sim no)
-		(at 212.344 79.248 0)
+		(at 210.82 77.978 0)
 		(effects
 			(font
@@
 	(text "IO7\n"
 		(exclude_from_sim no)
-		(at 213.36 99.568 0)
+		(at 212.852 99.568 0)
 		(effects
 			(font
@@
 	(text "IO2"
 		(exclude_from_sim no)
-		(at 213.36 86.868 0)
-		(effects
-			(font
-				(size 1.27 1.27)
-			)
+		(at 212.852 86.868 0)
+		(effects
+			(font
+				(size 1.27 1.27)
+			)
+		)
+	)
+	(text "Extremely weak pullup so that when the MCP3008 is\ndon't care, we can distinguish that from the 0 bit\nthat it intentionally sends."
+		(exclude_from_sim no)
+		(at 226.822 117.602 0)
+		(effects
+			(font
+				(size 1.27 1.27)
+			)
+			(justify left top)
 		)
 	)
@@
 	(text "IO4"
 		(exclude_from_sim no)
-		(at 213.36 91.948 0)
+		(at 212.852 91.948 0)
 		(effects
 			(font
@@
 	(text "IO1"
 		(exclude_from_sim no)
-		(at 213.36 84.328 0)
+		(at 212.852 84.328 0)
 		(effects
 			(font
@@
 	(text "IO0"
 		(exclude_from_sim no)
-		(at 213.36 81.788 0)
+		(at 212.852 81.788 0)
 		(effects
 			(font
@@
 	(text "NOTE\nprobably drop-in compatible with the MCP3208\nthat only gets 100ksps at 5V. no figure quoted for 3.3V"
 		(exclude_from_sim no)
-		(at 129.794 124.714 0)
+		(at 116.332 121.666 0)
 		(effects
 			(font
@@
 	)
 	(label "~{CS}"
-		(at 199.39 97.79 0)
+		(at 199.39 85.09 0)
 		(fields_autoplaced yes)
 		(effects
@@
 	)
 	(label "MISO"
-		(at 199.39 90.17 0)
+		(at 199.39 92.71 0)
 		(fields_autoplaced yes)
 		(effects
@@
 		)
 	)
+	(label "MISO"
+		(at 223.52 133.35 0)
+		(fields_autoplaced yes)
+		(effects
+			(font
+				(size 1.27 1.27)
+			)
+			(justify left bottom)
+		)
+	)
 	(label "AIN4N"
 		(at 96.52 96.52 180)
@@
 	)
 	(label "SCLK"
-		(at 199.39 92.71 0)
+		(at 199.39 90.17 0)
 		(fields_autoplaced yes)
 		(effects
@@
 	)
 	(label "MOSI"
-		(at 199.39 87.63 0)
+		(at 199.39 95.25 0)
 		(fields_autoplaced yes)
 		(effects
@@
 	(symbol
 		(lib_id "Connector_Generic:Conn_02x10_Odd_Even")
-		(at 220.98 90.17 0)
+		(at 220.98 92.71 0)
+		(mirror x)
 		(unit 1)
 		(exclude_from_sim no)
@@
 		(on_board yes)
 		(dnp no)
-		(fields_autoplaced yes)
 		(property "Reference" "J1"
-			(at 222.25 74.5955 0)
+			(at 222.25 76.962 0)
 			(effects
 				(font
@@
 		)
 		(property "Value" "Glasgow"
-			(at 222.25 77.0198 0)
+			(at 222.25 74.5377 0)
 			(effects
 				(font
@@
 		)
 		(property "Footprint" "Connector_PinHeader_2.54mm:PinHeader_2x10_P2.54mm_Vertical"
-			(at 220.98 90.17 0)
+			(at 220.98 92.71 0)
 			(effects
 				(font
@@
 		)
 		(property "Datasheet" "~"
-			(at 220.98 90.17 0)
+			(at 220.98 92.71 0)
 			(effects
 				(font
@@
 		)
 		(property "Description" "Generic connector, double row, 02x10, odd/even pin numbering scheme (row 1 odd numbers, row 2 even numbers), script generated (kicad-library-utils/schlib/autogen/connector/)"
-			(at 220.98 90.17 0)
+			(at 220.98 92.71 0)
 			(effects
 				(font
@@
 		)
 		(property "DigiKey" "SSW-110-03-T-D-ND"
-			(at 220.98 90.17 0)
+			(at 220.98 92.71 0)
 			(effects
 				(font
@@
 	)
 	(symbol
+		(lib_id "Device:R_Small_US")
+		(at 223.52 127 0)
+		(unit 1)
+		(exclude_from_sim no)
+		(in_bom yes)
+		(on_board yes)
+		(dnp no)
+		(fields_autoplaced yes)
+		(property "Reference" "R1"
+			(at 225.171 125.7878 0)
+			(effects
+				(font
+					(size 1.27 1.27)
+				)
+				(justify left)
+			)
+		)
+		(property "Value" "100k"
+			(at 225.171 128.2121 0)
+			(effects
+				(font
+					(size 1.27 1.27)
+				)
+				(justify left)
+			)
+		)
+		(property "Footprint" "Resistor_SMD:R_0805_2012Metric"
+			(at 223.52 127 0)
+			(effects
+				(font
+					(size 1.27 1.27)
+				)
+				(hide yes)
+			)
+		)
+		(property "Datasheet" "~"
+			(at 223.52 127 0)
+			(effects
+				(font
+					(size 1.27 1.27)
+				)
+				(hide yes)
+			)
+		)
+		(property "Description" "Resistor, small US symbol"
+			(at 223.52 127 0)
+			(effects
+				(font
+					(size 1.27 1.27)
+				)
+				(hide yes)
+			)
+		)
+		(pin "2"
+		)
+		(pin "1"
+		)
+		(instances
+			(project "mcp3008"
+				(path "/2788365e-935a-471c-aaba-4a57a0ad4aa0"
+					(reference "R1")
+					(unit 1)
+				)
+			)
+		)
+	)
+	(symbol
 		(lib_id "power:GND")
 		(at 204.47 50.8 0)
@@
 					(unit 1)
 				)
+			)
+		)
+	)
+	(symbol
+		(lib_id "power:VDD")
+		(at 223.52 121.92 0)
+		(unit 1)
+		(exclude_from_sim no)
+		(in_bom yes)
+		(on_board yes)
+		(dnp no)
+		(fields_autoplaced yes)
+		(property "Reference" "#PWR016"
+			(at 223.52 125.73 0)
+			(effects
+				(font
+					(size 1.27 1.27)
+				)
+				(hide yes)
+			)
+		)
+		(property "Value" "VDD"
+			(at 223.52 117.7869 0)
+			(effects
+				(font
+					(size 1.27 1.27)
+				)
+			)
+		)
+		(property "Footprint" ""
+			(at 223.52 121.92 0)
+			(effects
+				(font
+					(size 1.27 1.27)
+				)
+				(hide yes)
+			)
+		)
+		(property "Datasheet" ""
+			(at 223.52 121.92 0)
+			(effects
+				(font
+					(size 1.27 1.27)
+				)
+				(hide yes)
+			)
+		)
+		(property "Description" "Power symbol creates a global label with name \"VDD\""
+			(at 223.52 121.92 0)
+			(effects
+				(font
+					(size 1.27 1.27)
+				)
+				(hide yes)
+			)
+		)
+		(pin "1"
+		)
+		(instances
+			(project "mcp3008"
+				(path "/2788365e-935a-471c-aaba-4a57a0ad4aa0"
+					(reference "#PWR016")
+					(unit 1)
+				)
