File: resistor/resistor.kicad_pcb (KiCad board)
At the start: 4 copper layers, 63.5 x 37.5 mm, 25 parts, among them J1 ToADC, J2 Sensors, U3 MIC5366-2.0YC5-TR

Commit message: board revs, updated README
Connections:
- J1 pad 1: /VREF -> /S0
- J1 pad 10: /S4 -> /VREF
- J1 pad 11: /VREF -> /S5
- J1 pad 12: /S5 -> /VREF
- J1 pad 13: /VREF -> /S6
- J1 pad 14: /S6 -> /VREF
- J1 pad 15: /VREF -> /S7
- J1 pad 16: /S7 -> /VREF
- J1 pad 17: GND -> /VREF
- J1 pad 18: /VREF -> GND
- J1 pad 19: GND -> VAA
- J1 pad 2: /S0 -> /VREF
- J1 pad 20: VAA -> GND
- J1 pad 3: /VREF -> /S1
- J1 pad 4: /S1 -> /VREF
- J1 pad 5: /VREF -> /S2
- J1 pad 6: /S2 -> /VREF
- J1 pad 7: /VREF -> /S3
- J1 pad 8: /S3 -> /VREF
- J1 pad 9: /VREF -> /S4
Routing:
- net /VREF: track 88.0 -> 111.2 mm, vias 0 -> 1
- net /S0: track 57.6 -> 64.1 mm
- net /S7: track 53.2 -> 56.7 mm
- net /S5: track 51.1 -> 54.5 mm
- net /S3: track 51.3 -> 54.7 mm
- net /S4: track 63.2 -> 65.8 mm
- net /S6: track 65.8 -> 68.3 mm
- net /S2: track 61.7 -> 64.0 mm
- net /S1: track 57.6 -> 56.6 mm
- net VAA: vias 24 -> 26
- removed copper zone on F.Cu, net /VREF
Other:
- board text added: "Resistor Adapter rev1"
- board text removed: "Resistor Adapter rev0"
